File: Quadrotor.kicad_pcb (KiCad board)
At the start: 2 copper layers, 40 x 50 mm, 53 parts, among them J1 USB_C_Receptacle, J10 Conn_01x04_Male, J13 Conn_01x30_Male, J2 Conn_01x02_Male, J3 Conn_01x02_Male, J4 Conn_01x02_Male, J5 Conn_01x02_Male, J6 Conn_01x02_Male, J7 Conn_01x02_Male, J8 Conn_01x04_Male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

Commit message: 修改pcb文件
Parts:
- removed G***: LOGO, Logo:logo
