File: Quadrotor.sch (KiCad schematic (older format))
At the start: 52 parts, among them J1 USB_C_Receptacle, J10 Conn_01x04_Male, J13 Conn_01x30_Male, J2 Conn_01x02_Male, J3 Conn_01x02_Male, J4 Conn_01x02_Male, J5 Conn_01x02_Male, J6 Conn_01x02_Male, J7 Conn_01x02_Male, J8 Conn_01x04_Male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

Commit message: 修改pcb文件
Connections:
- no-connect marks 47 -> 54
Changed lines of the file:
@@
 NoConn ~ 7500 1100
 NoConn ~ 8000 2350
+NoConn ~ 7500 3000
+NoConn ~ 7500 3100
+NoConn ~ 7500 3200
+NoConn ~ 7500 4200
+NoConn ~ 7500 1400
+NoConn ~ 7500 1800
+NoConn ~ 7500 1600
 $EndSCHEMATC
